File: ESPHome-Thermostat-pcb.kicad_pcb (KiCad board)
At the start: 2 copper layers, 90 x 53 mm, 99 parts, among them J1 Si7021, J2 MT3608, J3 Relay_Out, J4 SSD1306_Display, J5 Vin, Q1 NMOS_YJL03N06A, Q10 PMOS_AP40P05, Q11 NMOS_YJL03N06A, Q12 PMOS_AP40P05, Q13 PMOS_AP40P05, Q14 NMOS_YJL03N06A, Q15 NMOS_YJL03N06A, Q16 PMOS_AP40P05, Q17 NMOS_YJL03N06A, Q18 PMOS_AP40P05, Q19 PMOS_AP40P05, Q2 NMOS_YJL03N06A, Q20 PMOS_AP40P05, Q3 PMOS_AP40P05, Q4 PMOS_AP40P05, Q5 NMOS_YJL03N06A, Q6 NMOS_YJL03N06A, Q7 PMOS_AP40P05, Q8 PMOS_AP40P05, Q9 NMOS_YJL03N06A, SW1 EC11_Rotary_Encoder_Switch, U1 NodeMCU_1.0_(ESP-12E), U2 PCF8574, U3 AMS1117-3.3

Commit message: development
Parts:
- removed Q13: PMOS_AP40P05, Package_TO_SOT_SMD:SOT-23
- added R46: 10K, Resistor_SMD:R_0805_2012Metric, F.Cu at (159.5, 92.2)
- R33: value 1M -> 2M
Connections:
- C1 pad 2: RESET -> Net-(C1-Pad2)
- Q14 pad 1: D1 -> Net-(C1-Pad2)
- Q14 pad 3: Net-(Q14-Pad3) -> RESET
- R33 pad 1: Net-(Q14-Pad3) -> Net-(C1-Pad2)
- R33 pad 2: RESET -> D1
Changed lines of the file:
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@@
   (net 79 "Net-(Q1-Pad3)")
   (net 80 "Net-(Q3-Pad1)")
-  (net 81 "Net-(Q14-Pad3)")
-  (net 82 "Net-(Q19-Pad1)")
-  (net 83 "Net-(J3-Pad1)")
+  (net 81 "Net-(Q19-Pad1)")
+  (net 82 "Net-(J3-Pad1)")
+  (net 83 "Net-(C1-Pad2)")
   (net_class Default "This is the default net class."
     (clearance 0.2)
@@
     (add_net GND)
     (add_net "Net-(BZ1-Pad1)")
+    (add_net "Net-(C1-Pad2)")
     (add_net "Net-(C3-Pad1)")
     (add_net "Net-(D1-Pad2)")
@@
     (add_net "Net-(Q11-Pad3)")
     (add_net "Net-(Q12-Pad1)")
-    (add_net "Net-(Q14-Pad3)")
     (add_net "Net-(Q15-Pad3)")
     (add_net "Net-(Q16-Pad1)")
@@
     (add_net Vout+)
   )
+  (module Resistor_SMD:R_0805_2012Metric (layer F.Cu)
+    (at 159.512 92.202)
+    (descr "Resistor SMD 0805 (2012 Metric), square (rectangular) end terminal, IPC_7351 nominal, (Body size source: IPC-SM-782 page 72, https://www.pcb-3d.com/wordpress/wp-content/uploads/ipc-sm-782a_amendment_1_and_2.pdf), generated with kicad-footprint-generator")
+    (tags resistor)
+    (attr smd)
+    (fp_text reference R46 (at 0 -1.65) (layer F.SilkS)
+      (effects (font (size 1 1) (thickness 0.15)))
+    )
+    (fp_text value 10K (at 0 1.65) (layer F.Fab)
+      (effects (font (size 1 1) (thickness 0.15)))
+    )
+    (fp_line (start 1.68 0.95) (end -1.68 0.95) (layer F.CrtYd) (width 0.05))
+    (fp_line (start 1.68 -0.95) (end 1.68 0.95) (layer F.CrtYd) (width 0.05))
+    (fp_line (start -1.68 -0.95) (end 1.68 -0.95) (layer F.CrtYd) (width 0.05))
+    (fp_line (start -1.68 0.95) (end -1.68 -0.95) (layer F.CrtYd) (width 0.05))
+    (fp_line (start -0.227064 0.735) (end 0.227064 0.735) (layer F.SilkS) (width 0.12))
+    (fp_line (start -0.227064 -0.735) (end 0.227064 -0.735) (layer F.SilkS) (width 0.12))
+    (fp_line (start 1 0.625) (end -1 0.625) (layer F.Fab) (width 0.1))
+    (fp_line (start 1 -0.625) (end 1 0.625) (layer F.Fab) (width 0.1))
+    (fp_line (start -1 -0.625) (end 1 -0.625) (layer F.Fab) (width 0.1))
+    (fp_line (start -1 0.625) (end -1 -0.625) (layer F.Fab) (width 0.1))
+    (fp_text user %R (at 0 0) (layer F.Fab)
+      (effects (font (size 0.5 0.5) (thickness 0.08)))
+    )
+    (pad 2 smd roundrect (at 0.9125 0) (size 1.025 1.4) (layers F.Cu F.Paste F.Mask) (roundrect_rratio 0.243902)
+      (net 20 +3.3V))
+    (pad 1 smd roundrect (at -0.9125 0) (size 1.025 1.4) (layers F.Cu F.Paste F.Mask) (roundrect_rratio 0.243902)
+      (net 69 RESET))
+    (model ${KISYS3DMOD}/Resistor_SMD.3dshapes/R_0805_2012Metric.wrl
+      (at (xyz 0 0 0))
+      (scale (xyz 1 1 1))
+      (rotate (xyz 0 0 0))
+    )
+  )
   (module Package_TO_SOT_SMD:SOT-23 (layer B.Cu)
     (at 53.086 51.816)
@@
       (net 20 +3.3V))
     (pad 2 smd rect (at -1 -0.95) (size 0.9 0.8) (layers B.Cu B.Paste B.Mask)
-      (net 83 "Net-(J3-Pad1)"))
+      (net 82 "Net-(J3-Pad1)"))
     (pad 1 smd rect (at -1 0.95) (size 0.9 0.8) (layers B.Cu B.Paste B.Mask)
       (net 19 GND))
@@
       (effects (font (size 1 1) (thickness 0.15)))
     )
-    (fp_text value 1M (at 0 1.65) (layer F.Fab)
+    (fp_text value 2M (at 0 1.65) (layer F.Fab)
       (effects (font (size 1 1) (thickness 0.15)))
     )
@@
     )
     (pad 2 smd roundrect (at 0.9125 0) (size 1.025 1.4) (layers F.Cu F.Paste F.Mask) (roundrect_rratio 0.243902)
-      (net 69 RESET))
+      (net 66 D1))
     (pad 1 smd roundrect (at -0.9125 0) (size 1.025 1.4) (layers F.Cu F.Paste F.Mask) (roundrect_rratio 0.243902)
-      (net 81 "Net-(Q14-Pad3)"))
+      (net 83 "Net-(C1-Pad2)"))
     (model ${KISYS3DMOD}/Resistor_SMD.3dshapes/R_0805_2012Metric.wrl
       (at (xyz 0 0 0))
@@
       (net 24 Vout+))
     (pad 1 smd roundrect (at -0.9125 0) (size 1.025 1.4) (layers F.Cu F.Paste F.Mask) (roundrect_rratio 0.243902)
-      (net 82 "Net-(Q19-Pad1)"))
+      (net 81 "Net-(Q19-Pad1)"))
     (model ${KISYS3DMOD}/Resistor_SMD.3dshapes/R_0805_2012Metric.wrl
       (at (xyz 0 0 0))
@@
       (net 65 "Net-(Q17-Pad3)"))
     (pad 1 smd roundrect (at -0.9125 0) (size 1.025 1.4) (layers F.Cu F.Paste F.Mask) (roundrect_rratio 0.243902)
-      (net 82 "Net-(Q19-Pad1)"))
+      (net 81 "Net-(Q19-Pad1)"))
     (model ${KISYS3DMOD}/Resistor_SMD.3dshapes/R_0805_2012Metric.wrl
       (at (xyz 0 0 0))
@@
     )
     (pad 2 smd roundrect (at 0.95 0) (size 1 1.45) (layers F.Cu F.Paste F.Mask) (roundrect_rratio 0.25)
-      (net 69 RESET))
+      (net 83 "Net-(C1-Pad2)"))
     (pad 1 smd roundrect (at -0.95 0) (size 1 1.45) (layers F.Cu F.Paste F.Mask) (roundrect_rratio 0.25)
       (net 19 GND))
@@
   )
   (module Package_TO_SOT_SMD:SOT-23 (layer F.Cu)
-    (at 120.326 30.36)
-    (descr "SOT-23, Standard")
-    (tags SOT-23)
-    (attr smd)
-    (fp_text reference Q13 (at 0 -2.5) (layer F.SilkS)
-      (effects (font (size 1 1) (thickness 0.15)))
-    )
-    (fp_text value PMOS_AP40P05 (at 0 2.5) (layer F.Fab)
-      (effects (font (size 1 1) (thickness 0.15)))
-    )
-    (fp_line (start 0.76 1.58) (end -0.7 1.58) (layer F.SilkS) (width 0.12))
-    (fp_line (start 0.76 -1.58) (end -1.4 -1.58) (layer F.SilkS) (width 0.12))
-    (fp_line (start -1.7 1.75) (end -1.7 -1.75) (layer F.CrtYd) (width 0.05))
-    (fp_line (start 1.7 1.75) (end -1.7 1.75) (layer F.CrtYd) (width 0.05))
-    (fp_line (start 1.7 -1.75) (end 1.7 1.75) (layer F.CrtYd) (width 0.05))
-    (fp_line (start -1.7 -1.75) (end 1.7 -1.75) (layer F.CrtYd) (width 0.05))
-    (fp_line (start 0.76 -1.58) (end 0.76 -0.65) (layer F.SilkS) (width 0.12))
-    (fp_line (start 0.76 1.58) (end 0.76 0.65) (layer F.SilkS) (width 0.12))
-    (fp_line (start -0.7 1.52) (end 0.7 1.52) (layer F.Fab) (width 0.1))
-    (fp_line (start 0.7 -1.52) (end 0.7 1.52) (layer F.Fab) (width 0.1))
-    (fp_line (start -0.7 -0.95) (end -0.15 -1.52) (layer F.Fab) (width 0.1))
-    (fp_line (start -0.15 -1.52) (end 0.7 -1.52) (layer F.Fab) (width 0.1))
-    (fp_line (start -0.7 -0.95) (end -0.7 1.5) (layer F.Fab) (width 0.1))
-    (fp_text user %R (at 0 0 90) (layer F.Fab)
-      (effects (font (size 0.5 0.5) (thickness 0.075)))
-    )
-    (pad 3 smd rect (at 1 0) (size 0.9 0.8) (layers F.Cu F.Paste F.Mask)
-      (net 69 RESET))
-    (pad 2 smd rect (at -1 0.95) (size 0.9 0.8) (layers F.Cu F.Paste F.Mask)
-      (net 20 +3.3V))
-    (pad 1 smd rect (at -1 -0.95) (size 0.9 0.8) (layers F.Cu F.Paste F.Mask)
-      (net 66 D1))
-    (model ${KISYS3DMOD}/Package_TO_SOT_SMD.3dshapes/SOT-23.wrl
-      (at (xyz 0 0 0))
-      (scale (xyz 1 1 1))
-      (rotate (xyz 0 0 0))
-    )
-  )
-  (module Package_TO_SOT_SMD:SOT-23 (layer F.Cu)
     (at 57.910001 43.050001)
     (descr "SOT-23, Standard")
@@
     )
     (pad 3 smd rect (at 1 0) (size 0.9 0.8) (layers F.Cu F.Paste F.Mask)
-      (net 81 "Net-(Q14-Pad3)"))
+      (net 69 RESET))
     (pad 2 smd rect (at -1 0.95) (size 0.9 0.8) (layers F.Cu F.Paste F.Mask)
       (net 19 GND))
     (pad 1 smd rect (at -1 -0.95) (size 0.9 0.8) (layers F.Cu F.Paste F.Mask)
-      (net 66 D1))
+      (net 83 "Net-(C1-Pad2)"))
     (model ${KISYS3DMOD}/Package_TO_SOT_SMD.3dshapes/SOT-23.wrl
       (at (xyz 0 0 0))
@@
       (net 24 Vout+))
     (pad 1 smd rect (at -1 -0.95) (size 0.9 0.8) (layers F.Cu F.Paste F.Mask)
-      (net 82 "Net-(Q19-Pad1)"))
+      (net 81 "Net-(Q19-Pad1)"))
     (model ${KISYS3DMOD}/Package_TO_SOT_SMD.3dshapes/SOT-23.wrl
       (at (xyz 0 0 0))
@@
       (net 22 Relay1))
     (pad 1 thru_hole rect (at 0 0 180) (size 2.6 2.6) (drill 1.3) (layers *.Cu *.Mask)
-      (net 83 "Net-(J3-Pad1)"))
+      (net 82 "Net-(J3-Pad1)"))
     (model ${KISYS3DMOD}/TerminalBlock_4Ucon.3dshapes/TerminalBlock_4Ucon_1x10_P3.50mm_Vertical.wrl
       (at (xyz 0 0 0))

Commit message: Development
Parts:
- removed the Q12 at (186.6, 51.0)
- removed the REF** at (136.8, 76.5)
- removed the REF** at (53.2, 76.5)
- added G***: LOGO, logo:d-diot-logo, F.Cu at (107.6, 85.6)
- added Q13: PMOS_AP40P05, Package_TO_SOT_SMD:SOT-23, F.Cu at (59.4, 74.4)
- added R40: 10K, Resistor_SMD:R_0805_2012Metric, F.Cu at (109.5, 95.9)
- added R41: 10K, Resistor_SMD:R_0805_2012Metric, F.Cu at (101.9, 96.0)
- added REF**: MountingHole_3.7mm, MountingHole:MountingHole_3.7mm, F.Cu at (136.8, 76.5)
- added REF**: MountingHole_3.7mm, MountingHole:MountingHole_3.7mm, F.Cu at (53.2, 76.5)
- D13: value D_Schottky -> SS14
- J1: footprint Connector_PinHeader_2.54mm:PinHeader_1x04_P2.54mm_Vertical -> Connector_PinSocket_2.54mm:PinSocket_1x04_P2.54mm_Vertical
- Q9: renamed from Q20; moved to F.Cu
- R42: renamed from R39; value 27K -> 7.5K
- moved R46 149.9 mm to (52.0, 92.3), turned to 180 degrees
- moved Q2 149.8 mm to (59.4, 88.3), turned to 270 degrees
- moved Q11 148.0 mm to (52.1, 69.5), turned to 90 degrees
- moved R22 142.8 mm to (51.3, 83.4), turned to 270 degrees
- moved Q7 142.5 mm to (55.8, 69.5), turned to 90 degrees
- moved R17 140.4 mm to (68.2, 98.7)
- moved R26 139.8 mm to (51.9, 101.9), turned to 180 degrees
- moved R13 139.2 mm to (57.4, 83.4), turned to 90 degrees
- moved R3 136.5 mm to (59.4, 83.4), turned to 270 degrees
- moved Q17 133.8 mm to (63.1, 88.3), turned to 270 degrees
- moved Q16 132.4 mm to (66.8, 69.5), turned to 90 degrees
- moved Q5 131.1 mm to (55.8, 88.3), turned to 270 degrees
- moved R4 129.9 mm to (61.5, 83.4), turned to 90 degrees
- moved R6 129.8 mm to (51.9, 95.5), turned to 180 degrees
- moved Q12 129.2 mm to (70.5, 88.3), turned to 270 degrees
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- renumbered J3 to J2, J2 to J3, Q9 to Q10, Q10 to Q11, Q11 to Q12, Q19 to Q18, Q18 to Q19, R46 to R34, R34 to R35, R35 to R36, R36 to R37, R37 to R38, R38 to R39, R40 to R43, R41 to R44, R42 to R45, R43 to R46, R44 to R47, R45 to R48
Connections:
- J5 pad 1: Net-(J5-Pad1) -> GND
- J5 pad 2: GND -> Net-(J5-Pad2)
- Q19 pad 2: Net-(J5-Pad1) -> Net-(J5-Pad2)
Routing:
- net +3.3V: track 0.00 -> 239.9 mm, vias 0 -> 8
- net Vout+: track 0.00 -> 234.8 mm, vias 0 -> 14
- net P0: track 0.00 -> 112.8 mm, vias 0 -> 3
- net D5-SCL: track 0.00 -> 98.5 mm, vias 0 -> 1
- net D4-SDA: track 0.00 -> 96.5 mm, vias 0 -> 1
- net P2: track 0.00 -> 90.7 mm, vias 0 -> 3
- net P6: track 0.00 -> 89.8 mm, vias 0 -> 4
- net P4: track 0.00 -> 87.0 mm, vias 0 -> 2
- net D1: track 0.00 -> 79.5 mm, vias 0 -> 2
- net P1: track 0.00 -> 75.5 mm, vias 0 -> 3
- net D6: track 0.00 -> 60.4 mm, vias 0 -> 2
- net P3: track 0.00 -> 58.8 mm, vias 0 -> 3
- net D7: track 0.00 -> 48.4 mm, vias 0 -> 2
- net D2: track 0.00 -> 48.3 mm
- net P7: track 0.00 -> 31.6 mm, vias 0 -> 1
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- added copper zone on B.Cu, net GND
- added copper zone on F.Cu, net GND
Other:
- rule via_min_drill: 0.3 -> 0.35
- rule via_min_size: 0.4 -> 0.65
- board text added: "+"
- board text added: "+3.3V"
- board text added: "ESPHome Thermostat pcb - v.1.0"
- board text added: "GND"
- board text added: "SCL"
- board text added: "SDA"
- board text added: "V+"
- board text added: "VDD"

Commit message: Release board v.1.0
Parts:
- moved J1 7.88 mm to (79.8, 100.8), turned to 90 degrees
Routing:
- net P0: track 112.8 -> 121.9 mm, vias 3 -> 4
- net P6: track 89.8 -> 93.5 mm, vias 4 -> 6
- net D5-SCL: track 98.5 -> 95.2 mm
- net +3.3V: track 239.9 -> 237.0 mm
- net GND: track 7.40 -> 8.62 mm, vias 18 -> 20
- net D4-SDA: track 96.5 -> 97.7 mm

Commit message: Development v.2.0
Parts:
- removed R16, R17, R26, R27, R37, R46, R5, R6: 10K, Resistor_SMD:R_0805_2012Metric
- added Q20: NMOS_YJL03N06A, Package_TO_SOT_SMD:SOT-23, B.Cu at (130.6, 61.5)
- added Q21: NMOS_YJL03N06A, Package_TO_SOT_SMD:SOT-23, B.Cu at (59.4, 83.0)
- added Q22: NMOS_YJL03N06A, Package_TO_SOT_SMD:SOT-23, B.Cu at (126.5, 101.1)
- added Q23: NMOS_YJL03N06A, Package_TO_SOT_SMD:SOT-23, B.Cu at (59.2, 59.7)
- added Q24: NMOS_YJL03N06A, Package_TO_SOT_SMD:SOT-23, B.Cu at (68.1, 94.5)
- added Q25: NMOS_YJL03N06A, Package_TO_SOT_SMD:SOT-23, B.Cu at (130.6, 71.3)
- added Q26: NMOS_YJL03N06A, Package_TO_SOT_SMD:SOT-23, B.Cu at (59.2, 69.3)
- added Q27: NMOS_YJL03N06A, Package_TO_SOT_SMD:SOT-23, B.Cu at (131.1, 82.0)
- moved J1 17.0 mm to (90.4, 87.6), turned to 180 degrees
- turned R18 to 180 degrees
Connections:
- D10 pad 1: GND -> Net-(D10-Pad1)
- D12 pad 1: GND -> Net-(D12-Pad1)
- D14 pad 1: GND -> Net-(D14-Pad1)
- D16 pad 1: GND -> Net-(D16-Pad1)
- D2 pad 1: GND -> Net-(D2-Pad1)
- D4 pad 1: GND -> Net-(D4-Pad1)
- D7 pad 1: GND -> Net-(D7-Pad1)
- D8 pad 1: GND -> Net-(D8-Pad1)
- R18 pad 1: P6 -> Net-(D7-Pad2)
- R18 pad 2: Net-(D7-Pad2) -> +3.3V
- R19 pad 1: P1 -> +3.3V
- R28 pad 1: P7 -> +3.3V
- R29 pad 1: P2 -> +3.3V
- R38 pad 1: P3 -> +3.3V
- R47 pad 1: P4 -> +3.3V
- R7 pad 1: P0 -> +3.3V
- R8 pad 1: P5 -> +3.3V
Routing:
- net +3.3V: track 237.0 -> 362.0 mm, vias 8 -> 13
- net P3: track 58.8 -> 77.3 mm
- net D4-SDA: track 97.7 -> 113.6 mm
- net P0: track 121.9 -> 110.8 mm, vias 4 -> 3
- net P4: track 87.0 -> 94.0 mm, vias 2 -> 4
- net Net-(D2-Pad1): track 0.00 -> 6.92 mm
- net Net-(D7-Pad1): track 0.00 -> 6.50 mm
- net P2: track 90.7 -> 97.1 mm
- net Net-(D8-Pad1): track 0.00 -> 5.38 mm
- net Net-(D12-Pad1): track 0.00 -> 5.37 mm
- net Net-(D16-Pad1): track 0.00 -> 5.22 mm
- net Net-(D4-Pad1): track 0.00 -> 5.12 mm
- net Net-(D14-Pad1): track 0.00 -> 4.75 mm
- net P5: track 18.6 -> 14.0 mm
- net P7: track 31.6 -> 26.9 mm
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Other:
- board text added: "ESPHome Thermostat pcb - v.2.0"
- board text removed: "ESPHome Thermostat pcb - v.1.0"
