File: ESPHome-Thermostat-pcb.sch (KiCad schematic (older format))
At the start: 97 parts, among them J1 Si7021, J2 MT3608, J3 Relay_Out, J4 SSD1306_Display, J5 Vin, Q1 NMOS_YJL03N06A, Q10 PMOS_AP40P05, Q11 NMOS_YJL03N06A, Q12 PMOS_AP40P05, Q13 PMOS_AP40P05, Q14 NMOS_YJL03N06A, Q15 NMOS_YJL03N06A, Q16 PMOS_AP40P05, Q17 NMOS_YJL03N06A, Q18 PMOS_AP40P05, Q19 PMOS_AP40P05, Q2 NMOS_YJL03N06A, Q20 PMOS_AP40P05, Q3 PMOS_AP40P05, Q4 PMOS_AP40P05, Q5 NMOS_YJL03N06A, Q6 NMOS_YJL03N06A, Q7 PMOS_AP40P05, Q8 PMOS_AP40P05, Q9 NMOS_YJL03N06A, SW1 EC11_Rotary_Encoder_Switch, U1 NodeMCU_1.0_(ESP-12E), U2 PCF8574, U3 AMS1117-3.3

Commit message: development
Parts:
- removed Q13: PMOS_AP40P05, Package_TO_SOT_SMD:SOT-23, symbol Device:Q_PMOS_GSD
- added R46: 10K, Resistor_SMD:R_0805_2012Metric, symbol Device:R
- R33: value 1M -> 2M
Connections:
- net +3.3V: now also R46.2
- net D1: now also R33.2; no longer Q14.1 (G)
- net RESET: now also Q14.3 (D), R46.1; no longer C1.2, R33.2
- net at R33.1: now also C1.2, Q14.1 (G); no longer Q14.3 (D)
Other:
- moved on the sheet: C1, Q14, R33
Changed lines of the file:
@@
 L Device:Q_NMOS_GSD Q14
 U 1 1 61CAFC02
-P 7750 2400
-F 0 "Q14" H 7955 2446 50  0000 L CNN
-F 1 "NMOS_YJL03N06A" H 7955 2355 50  0000 L CNN
-F 2 "Package_TO_SOT_SMD:SOT-23" H 7950 2500 50  0001 C CNN
-F 3 "~" H 7750 2400 50  0001 C CNN
-	1    7750 2400
-	0    -1   -1   0
+P 6900 2450
+F 0 "Q14" H 7105 2496 50  0000 L CNN
+F 1 "NMOS_YJL03N06A" H 7105 2405 50  0000 L CNN
+F 2 "Package_TO_SOT_SMD:SOT-23" H 7100 2550 50  0001 C CNN
+F 3 "~" H 6900 2450 50  0001 C CNN
+	1    6900 2450
+	1    0    0    -1
 $EndComp
 Wire Wire Line
@@
 Text GLabel 850  2250 0    50   Input ~ 0
 RESET
-$Comp
-L Device:Q_PMOS_GSD Q13
-U 1 1 61E18905
-P 6700 2200
-F 0 "Q13" V 6949 2200 50  0000 C CNN
-F 1 "PMOS_AP40P05" V 7040 2200 50  0000 C CNN
-F 2 "Package_TO_SOT_SMD:SOT-23" H 6900 2300 50  0001 C CNN
-F 3 "~" H 6700 2200 50  0001 C CNN
-	1    6700 2200
-	0    1    1    0
-$EndComp
-Text GLabel 6500 2300 0    50   Input ~ 0
-+3.3V
-Connection ~ 6700 1750
-Wire Wire Line
-	7100 2300 6900 2300
+Text GLabel 7000 1750 2    50   Input ~ 0
++3.3V
 $Comp
 L power:GND #PWR036
 U 1 1 61E9C208
-P 7100 2600
-F 0 "#PWR036" H 7100 2350 50  0001 C CNN
-F 1 "GND" V 7105 2472 50  0000 R CNN
-F 2 "" H 7100 2600 50  0001 C CNN
-F 3 "" H 7100 2600 50  0001 C CNN
-	1    7100 2600
-	1    0    0    -1
-$EndComp
-Text GLabel 7100 2200 1    50   Input ~ 0
+P 6400 2350
+F 0 "#PWR036" H 6400 2100 50  0001 C CNN
+F 1 "GND" V 6405 2222 50  0000 R CNN
+F 2 "" H 6400 2350 50  0001 C CNN
+F 3 "" H 6400 2350 50  0001 C CNN
+	1    6400 2350
+	0    1    1    0
+$EndComp
+Text GLabel 7100 2200 2    50   Input ~ 0
 RESET
-Wire Wire Line
-	7100 2200 7100 2300
-Connection ~ 7100 2300
 $Comp
 L Device:R R33
 U 1 1 61E9FC38
-P 7400 2300
-F 0 "R33" V 7193 2300 50  0000 C CNN
-F 1 "1M" V 7284 2300 50  0000 C CNN
-F 2 "Resistor_SMD:R_0805_2012Metric" V 7330 2300 50  0001 C CNN
-F 3 "~" H 7400 2300 50  0001 C CNN
-	1    7400 2300
-	0    1    1    0
-$EndComp
-Wire Wire Line
-	7250 2300 7100 2300
+P 6700 2050
+F 0 "R33" V 6493 2050 50  0000 C CNN
+F 1 "2M" V 6584 2050 50  0000 C CNN
+F 2 "Resistor_SMD:R_0805_2012Metric" V 6630 2050 50  0001 C CNN
+F 3 "~" H 6700 2050 50  0001 C CNN
+	1    6700 2050
+	-1   0    0    1
+$EndComp
 $Comp
 L power:GND #PWR038
 U 1 1 61EADD37
-P 7950 2300
-F 0 "#PWR038" H 7950 2050 50  0001 C CNN
-F 1 "GND" V 7955 2172 50  0000 R CNN
-F 2 "" H 7950 2300 50  0001 C CNN
-F 3 "" H 7950 2300 50  0001 C CNN
-	1    7950 2300
-	0    -1   -1   0
-$EndComp
-Wire Wire Line
-	6700 1750 6700 1900
-Wire Wire Line
-	7750 2600 7750 2900
-Wire Wire Line
-	7750 2900 6050 2900
-Wire Wire Line
-	6050 2900 6050 1900
-Wire Wire Line
-	6050 1900 6700 1900
-Connection ~ 6700 1900
-Wire Wire Line
-	6700 1900 6700 2000
+P 7000 2650
+F 0 "#PWR038" H 7000 2400 50  0001 C CNN
+F 1 "GND" V 7005 2522 50  0000 R CNN
+F 2 "" H 7000 2650 50  0001 C CNN
+F 3 "" H 7000 2650 50  0001 C CNN
+	1    7000 2650
+	1    0    0    -1
+$EndComp
 Wire Wire Line
 	2050 5200 2100 5200
@@
 L Device:C C1
 U 1 1 61D298D5
-P 7100 2450
-F 0 "C1" H 7215 2496 50  0000 L CNN
-F 1 "10uF" H 7215 2405 50  0000 L CNN
-F 2 "Capacitor_SMD:C_0805_2012Metric" H 7138 2300 50  0001 C CNN
-F 3 "~" H 7100 2450 50  0001 C CNN
-	1    7100 2450
-	-1   0    0    1
+P 6550 2350
+F 0 "C1" H 6665 2396 50  0000 L CNN
+F 1 "10uF" H 6665 2305 50  0000 L CNN
+F 2 "Capacitor_SMD:C_0805_2012Metric" H 6588 2200 50  0001 C CNN
+F 3 "~" H 6550 2350 50  0001 C CNN
+	1    6550 2350
+	0    -1   -1   0
 $EndComp
 Text GLabel 5000 1950 2    50   Input ~ 0
@@
 Wire Wire Line
 	5000 1850 5000 1950
+Wire Wire Line
+	6700 1900 6700 1750
+Connection ~ 6700 1750
+Wire Wire Line
+	6700 2200 6700 2350
+Connection ~ 6700 2350
+Wire Wire Line
+	6700 2350 6700 2450
+$Comp
+L Device:R R46
+U 1 1 61DFB003
+P 7000 2000
+F 0 "R46" V 6793 2000 50  0000 C CNN
+F 1 "10K" V 6884 2000 50  0000 C CNN
+F 2 "Resistor_SMD:R_0805_2012Metric" V 6930 2000 50  0001 C CNN
+F 3 "~" H 7000 2000 50  0001 C CNN
+	1    7000 2000
+	-1   0    0    1
+$EndComp
+Wire Wire Line
+	7000 1850 7000 1750
+Wire Wire Line
+	7000 2150 7000 2200
+Wire Wire Line
+	7100 2200 7000 2200
+Connection ~ 7000 2200
+Wire Wire Line
+	7000 2200 7000 2250
 $EndSCHEMATC

Commit message: Development
Parts:
- added R40, R41: 10K, Resistor_SMD:R_0805_2012Metric, symbol Device:R
- BZ1: Description (none) -> Universal Passive Buzzer; Link (none) -> https://www.ebay.it/itm/5PCS-Universal-Passive-Buzzer-16-oh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; MOQ (none) -> 5; MPN (none) -> NA; Manufacturer (none) -> NA; Price (none) -> 0.25; VPN (none) -> NA; Vendor (none) -> Ebay
- C1, C3: Description (none) -> Capacitor 10 uF SMD 0805; Link (none) -> https://lcsc.com/product-detail/Multilayer-Ceramic-Capacito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; MOQ (none) -> 50; MPN (none) -> CL21A106KAYNNNE; Manufacturer (none) -> Samsung Electro-Mechanics; Price (none) -> 0.0076; VPN (none) -> C15850; Vendor (none) -> LCSC
- C2: Description (none) -> Capacitor 22uF Tantalum SMD; Link (none) -> https://lcsc.com/product-detail/Tantalum-Capacitors_AVX_TAJ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; MOQ (none) -> 1; MPN (none) -> TAJB226M016RNJ; Manufacturer (none) -> AVX; Price (none) -> 0.13; VPN (none) -> C24518; Vendor (none) -> LCSC
- D1, D11, D15, D3, D5, D6, D9: Description (none) -> Schottky Barrier Diodes 40V 1A SMD DO-214AC/SMA; Link (none) -> https://lcsc.com/product-detail/Schottky-Barrier-Diodes-SBD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; MOQ (none) -> 20; MPN (none) -> SS14; Manufacturer (none) -> MDD（Microdiode Electronics); Price (none) -> 0.018; VPN (none) -> C2480; Vendor (none) -> LCSC
- D10, D14, D4, D7: Description (none) -> Yellow Led SMD 0805; Link (none) -> https://lcsc.com/product-detail/Light-Emitting-Diodes-LED_Y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; MOQ (none) -> 50; MPN (none) -> NCD0805Y1; Manufacturer (none) -> Foshan NationStar; Price (none) -> 0.019; VPN (none) -> C84261; Vendor (none) -> LCSC
- D12: Description (none) -> White Led SMD 0805; Link (none) -> https://lcsc.com/product-detail/Light-Emitting-Diodes-LED_Y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; MOQ (none) -> 50; MPN (none) -> SZYY0805W; Manufacturer (none) -> Yongyu Photoelectric; Price (none) -> 0.012; VPN (none) -> C434434; Vendor (none) -> LCSC
- D13: value D_Schottky -> SS14; Description (none) -> Schottky Barrier Diodes 40V 1A SMD DO-214AC/SMA; Link (none) -> https://lcsc.com/product-detail/Schottky-Barrier-Diodes-SBD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; MOQ (none) -> 20; MPN (none) -> SS14; Manufacturer (none) -> MDD（Microdiode Electronics); Price (none) -> 0.018; VPN (none) -> C2480; Vendor (none) -> LCSC
- D16: Description (none) -> Green Led SMD 0805; Link (none) -> https://lcsc.com/product-detail/Light-Emitting-Diodes-LED_Y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; MOQ (none) -> 20; MPN (none) -> NCD0805G1; Manufacturer (none) -> Foshan NationStar Optoelectronics; Price (none) -> 0.021; VPN (none) -> C84260; Vendor (none) -> LCSC
- D2: Description (none) -> Red Led SMD 0805; Link (none) -> https://lcsc.com/product-detail/Light-Emitting-Diodes-LED_L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; MPN (none) -> BL-HUE35A-AV-TRE; Manufacturer (none) -> BrtLed(Bright LED Elec); VPN (none) -> C138549; Vendor (none) -> LCSC
- D8: Description (none) -> Blu Led SMD 0805; Link (none) -> https://lcsc.com/product-detail/Light-Emitting-Diodes-LED_B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; MOQ (none) -> 20; MPN (none) -> NCD0805B2; Manufacturer (none) -> Foshan NationStar; Price (none) -> 0.021; VPN (none) -> C84259; Vendor (none) -> LCSC
- J1: footprint Connector_PinHeader_2.54mm:PinHeader_1x04_P2.54mm_Vertical -> Connector_PinSocket_2.54mm:PinSocket_1x04_P2.54mm_Vertical; Description (none) -> Pin header female 1×04 p.2.54 mm; Link (none) -> NA; MOQ (none) -> NA; MPN (none) -> NA; Manufacturer (none) -> NA; Price (none) -> NA; VPN (none) -> NA; Vendor (none) -> NA
- J2: renamed from J3; Description (none) -> Pluggable terminal block 1x10 p.3.5 mm straight needle; Link (none) -> https://it.aliexpress.com/item/1005002951707517.html?spm=a2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; MOQ (none) -> NA; MPN (none) -> NA; Manufacturer (none) -> KF2EDG; Price (none) -> NA; VPN (none) -> NA; Vendor (none) -> Aliexpress
- J3: renamed from J2; Description (none) -> Step-up boost converter MT3608 module; Link (none) -> https://it.aliexpress.com/item/1005002433903674.html?spm=a2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; MOQ (none) -> 1; MPN (none) -> NA; Manufacturer (none) -> NA; Price (none) -> 0.45; VPN (none) -> NA; Vendor (none) -> Aliexpress
- J4: Description (none) -> Pin header female 1×04 p.2.54 mm; Link (none) -> NA; MOQ (none) -> NA; MPN (none) -> NA; Manufacturer (none) -> NA; Price (none) -> NA; VPN (none) -> NA; Vendor (none) -> NA
- J5: Description (none) -> Pluggable terminal block 1x02 p.3.5 mm straight needle; Link (none) -> https://it.aliexpress.com/item/1005002951707517.html?spm=a2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; MOQ (none) -> NA; MPN (none) -> NA; Manufacturer (none) -> KF2EDG; Price (none) -> NA; VPN (none) -> NA; Vendor (none) -> Aliexpress
- JP1, JP2, JP3: Description (none) -> Solder Jumper pad (no components required); Link (none) -> NA; MOQ (none) -> NA; MPN (none) -> NA; Manufacturer (none) -> NA; Price (none) -> NA; VPN (none) -> NA; Vendor (none) -> NA
- Q1, Q14, Q15, Q17, Q2, Q5, Q6: Description (none) -> N-Channel mosfet 60V 3A RDS ON 86mΩ, Gate threshold 1.3V SM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; Link (none) -> https://lcsc.com/product-detail/MOSFETs_Yangzhou-Yangjie-El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; MOQ (none) -> 10; MPN (none) -> YJL03N06A; Manufacturer (none) -> Yangzhou Yangjie Elec Tech; Price (none) -> 0.038; VPN (none) -> C699294; Vendor (none) -> LCSC
- Q10: renamed from Q9; Description (none) -> N-Channel mosfet 60V 3A RDS ON 86mΩ, Gate threshold 1.3V SM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; Link (none) -> https://lcsc.com/product-detail/MOSFETs_Yangzhou-Yangjie-El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; MOQ (none) -> 10; MPN (none) -> YJL03N06A; Manufacturer (none) -> Yangzhou Yangjie Elec Tech; Price (none) -> 0.038; VPN (none) -> C699294; Vendor (none) -> LCSC
- Q11: renamed from Q10; Description (none) -> P-Channel mosfet 40V 5A RDS ON 65mΩ, Gate threshold -1.6V S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; Link (none) -> https://lcsc.com/product-detail/MOSFETs_ALLPOWER-ShenZhen-Q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; MOQ (none) -> 10; MPN (none) -> AP40P05; Manufacturer (none) -> ALLPOWER(ShenZhen Quan Li Semiconductor); Price (none) -> 0.033; VPN (none) -> C2886385; Vendor (none) -> LCSC
- Q12: renamed from Q11; Description (none) -> N-Channel mosfet 60V 3A RDS ON 86mΩ, Gate threshold 1.3V SM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; Link (none) -> https://lcsc.com/product-detail/MOSFETs_Yangzhou-Yangjie-El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; MOQ (none) -> 10; MPN (none) -> YJL03N06A; Manufacturer (none) -> Yangzhou Yangjie Elec Tech; Price (none) -> 0.038; VPN (none) -> C699294; Vendor (none) -> LCSC
- Q13: renamed from Q12; Description (none) -> P-Channel mosfet 40V 5A RDS ON 65mΩ, Gate threshold -1.6V S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; Link (none) -> https://lcsc.com/product-detail/MOSFETs_ALLPOWER-ShenZhen-Q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; MOQ (none) -> 10; MPN (none) -> AP40P05; Manufacturer (none) -> ALLPOWER(ShenZhen Quan Li Semiconductor); Price (none) -> 0.033; VPN (none) -> C2886385; Vendor (none) -> LCSC
- Q16, Q3, Q4, Q7, Q8: Description (none) -> P-Channel mosfet 40V 5A RDS ON 65mΩ, Gate threshold -1.6V S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; Link (none) -> https://lcsc.com/product-detail/MOSFETs_ALLPOWER-ShenZhen-Q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; MOQ (none) -> 10; MPN (none) -> AP40P05; Manufacturer (none) -> ALLPOWER(ShenZhen Quan Li Semiconductor); Price (none) -> 0.033; VPN (none) -> C2886385; Vendor (none) -> LCSC
- Q18: renamed from Q19; Description (none) -> P-Channel mosfet 40V 5A RDS ON 65mΩ, Gate threshold -1.6V S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; Link (none) -> https://lcsc.com/product-detail/MOSFETs_ALLPOWER-ShenZhen-Q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; MOQ (none) -> 10; MPN (none) -> AP40P05; Manufacturer (none) -> ALLPOWER(ShenZhen Quan Li Semiconductor); Price (none) -> 0.033; VPN (none) -> C2886385; Vendor (none) -> LCSC
- Q19: renamed from Q18; Description (none) -> P-Channel mosfet 40V 5A RDS ON 65mΩ, Gate threshold -1.6V S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; Link (none) -> https://lcsc.com/product-detail/MOSFETs_ALLPOWER-ShenZhen-Q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; MOQ (none) -> 10; MPN (none) -> AP40P05; Manufacturer (none) -> ALLPOWER(ShenZhen Quan Li Semiconductor); Price (none) -> 0.033; VPN (none) -> C2886385; Vendor (none) -> LCSC
- Q9: renamed from Q20; Description (none) -> P-Channel mosfet 40V 5A RDS ON 65mΩ, Gate threshold -1.6V S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; Link (none) -> https://lcsc.com/product-detail/MOSFETs_ALLPOWER-ShenZhen-Q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; MOQ (none) -> 10; MPN (none) -> AP40P05; Manufacturer (none) -> ALLPOWER(ShenZhen Quan Li Semiconductor); Price (none) -> 0.033; VPN (none) -> C2886385; Vendor (none) -> LCSC
- R1, R12, R13, R14, R15, R16, R17, R2, R22, R23, R24, R25, R26, R27, R3, R32, R4, R5, R6: Description (none) -> Resistor 10K SMD 0805; Link (none) -> https://lcsc.com/product-detail/High-Precision-Low-TCR-SMD-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; MOQ (none) -> 50; MPN (none) -> TC0550F1002T5E; Manufacturer (none) -> UNI-ROYAL(Uniroyal Elec); Price (none) -> 0.007; VPN (none) -> C57859; Vendor (none) -> LCSC
- R10, R20, R21, R30, R31, R9: Description (none) -> Resistor 1M SMD 0805; Link (none) -> https://lcsc.com/product-detail/Chip-Resistor-Surface-Mount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; MOQ (none) -> 50; MPN (none) -> TC0525F1004T5E; Manufacturer (none) -> UNI-ROYAL(Uniroyal Elec); Price (none) -> 0.009; VPN (none) -> C75782; Vendor (none) -> LCSC
- R11, R18, R19, R28, R29, R7, R8: Description (none) -> Resistor 300 Ohm SMD 0805; Link (none) -> https://lcsc.com/product-detail/High-Precision-Low-TCR-SMD-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; MOQ (none) -> 50; MPN (none) -> TC0525F3000T5E; Manufacturer (none) -> UNI-ROYAL(Uniroyal Elec); Price (none) -> 0.008; VPN (none) -> C61685; Vendor (none) -> LCSC
- R33: Description (none) -> Resistor 2M SMD 0805; Link (none) -> https://lcsc.com/product-detail/Chip-Resistor-Surface-Mount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; MOQ (none) -> 100; MPN (none) -> FRC0805J205 TS; Manufacturer (none) -> FOJAN; Price (none) -> 0.0015; VPN (none) -> C2907316; Vendor (none) -> LCSC
- R34: renamed from R46; Description (none) -> Resistor 10K SMD 0805; Link (none) -> https://lcsc.com/product-detail/High-Precision-Low-TCR-SMD-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; MOQ (none) -> 50; MPN (none) -> TC0550F1002T5E; Manufacturer (none) -> UNI-ROYAL(Uniroyal Elec); Price (none) -> 0.007; VPN (none) -> C57859; Vendor (none) -> LCSC
- R35: renamed from R34; Description (none) -> Resistor 10K SMD 0805; Link (none) -> https://lcsc.com/product-detail/High-Precision-Low-TCR-SMD-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; MOQ (none) -> 50; MPN (none) -> TC0550F1002T5E; Manufacturer (none) -> UNI-ROYAL(Uniroyal Elec); Price (none) -> 0.007; VPN (none) -> C57859; Vendor (none) -> LCSC
- R36: renamed from R35; Description (none) -> Resistor 10K SMD 0805; Link (none) -> https://lcsc.com/product-detail/High-Precision-Low-TCR-SMD-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; MOQ (none) -> 50; MPN (none) -> TC0550F1002T5E; Manufacturer (none) -> UNI-ROYAL(Uniroyal Elec); Price (none) -> 0.007; VPN (none) -> C57859; Vendor (none) -> LCSC
- R37: renamed from R36; Description (none) -> Resistor 10K SMD 0805; Link (none) -> https://lcsc.com/product-detail/High-Precision-Low-TCR-SMD-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; MOQ (none) -> 50; MPN (none) -> TC0550F1002T5E; Manufacturer (none) -> UNI-ROYAL(Uniroyal Elec); Price (none) -> 0.007; VPN (none) -> C57859; Vendor (none) -> LCSC
- R38: renamed from R37; Description (none) -> Resistor 300 Ohm SMD 0805; Link (none) -> https://lcsc.com/product-detail/High-Precision-Low-TCR-SMD-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; MOQ (none) -> 50; MPN (none) -> TC0525F3000T5E; Manufacturer (none) -> UNI-ROYAL(Uniroyal Elec); Price (none) -> 0.008; VPN (none) -> C61685; Vendor (none) -> LCSC
- R39: renamed from R38; Description (none) -> Resistor 1M SMD 0805; Link (none) -> https://lcsc.com/product-detail/Chip-Resistor-Surface-Mount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; MOQ (none) -> 50; MPN (none) -> TC0525F1004T5E; Manufacturer (none) -> UNI-ROYAL(Uniroyal Elec); Price (none) -> 0.009; VPN (none) -> C75782; Vendor (none) -> LCSC
- R42: renamed from R39; value 27K -> 7.5K; Description (none) -> Resistor 7.5K SMD 0805; Link (none) -> https://lcsc.com/product-detail/Chip-Resistor-Surface-Mount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; MOQ (none) -> 50; MPN (none) -> 0805W8D7501T5E; Manufacturer (none) -> UNI-ROYAL(Uniroyal Elec); Price (none) -> 0.007; VPN (none) -> C422815; Vendor (none) -> LCSC
- R43: renamed from R40; Description (none) -> Resistor 1K SMD 0805; Link (none) -> https://lcsc.com/product-detail/Chip-Resistor-Surface-Mount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; MOQ (none) -> 50; MPN (none) -> 0805W8D1001T5E; Manufacturer (none) -> UNI-ROYAL(Uniroyal Elec); Price (none) -> 0.0065; VPN (none) -> C2767302; Vendor (none) -> LCSC
- R44: renamed from R41; Description (none) -> Resistor 10K SMD 0805; Link (none) -> https://lcsc.com/product-detail/High-Precision-Low-TCR-SMD-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; MOQ (none) -> 50; MPN (none) -> TC0550F1002T5E; Manufacturer (none) -> UNI-ROYAL(Uniroyal Elec); Price (none) -> 0.007; VPN (none) -> C57859; Vendor (none) -> LCSC
- R45: renamed from R42; Description (none) -> Resistor 10K SMD 0805; Link (none) -> https://lcsc.com/product-detail/High-Precision-Low-TCR-SMD-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; MOQ (none) -> 50; MPN (none) -> TC0550F1002T5E; Manufacturer (none) -> UNI-ROYAL(Uniroyal Elec); Price (none) -> 0.007; VPN (none) -> C57859; Vendor (none) -> LCSC
- R46: renamed from R43; Description (none) -> Resistor 10K SMD 0805; Link (none) -> https://lcsc.com/product-detail/High-Precision-Low-TCR-SMD-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; MOQ (none) -> 50; MPN (none) -> TC0550F1002T5E; Manufacturer (none) -> UNI-ROYAL(Uniroyal Elec); Price (none) -> 0.007; VPN (none) -> C57859; Vendor (none) -> LCSC
- R47: renamed from R44; Description (none) -> Resistor 300 Ohm SMD 0805; Link (none) -> https://lcsc.com/product-detail/High-Precision-Low-TCR-SMD-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; MOQ (none) -> 50; MPN (none) -> TC0525F3000T5E; Manufacturer (none) -> UNI-ROYAL(Uniroyal Elec); Price (none) -> 0.008; VPN (none) -> C61685; Vendor (none) -> LCSC
- R48: renamed from R45; Description (none) -> Resistor 1M SMD 0805; Link (none) -> https://lcsc.com/product-detail/Chip-Resistor-Surface-Mount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; MOQ (none) -> 50; MPN (none) -> TC0525F1004T5E; Manufacturer (none) -> UNI-ROYAL(Uniroyal Elec); Price (none) -> 0.009; VPN (none) -> C75782; Vendor (none) -> LCSC
- SW1: Description (none) -> EC11 Rotary encoder with push button - 15 mm shaft S; Link (none) -> https://www.ebay.it/itm/182373237976; MOQ (none) -> 10; MPN (none) -> EC11; Manufacturer (none) -> Alpsalpine; Price (none) -> 0.57; VPN (none) -> NA; Vendor (none) -> Ebay
- U1: Description (none) -> 2 x Pin header female 1×15 p.2.54 mm; Link (none) -> NA; MOQ (none) -> NA; MPN (none) -> NA; Manufacturer (none) -> NA; Price (none) -> NA; VPN (none) -> NA; Vendor (none) -> NA
- U2: Description (none) -> Remote 8 bit I/O expander for I2C bus PCF8574T SMD SOIC-16; Link (none) -> https://lcsc.com/product-detail/I-O-Expanders_NXP-Semicon-P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; MOQ (none) -> 1; MPN (none) -> PCF8574T/3,518; Manufacturer (none) -> NXP Semicon; Price (none) -> 1.17; VPN (none) -> C7605; Vendor (none) -> LCSC
- U3: Description (none) -> AMS1117 3.3V voltage regulator SMD SOT-223; Link (none) -> https://lcsc.com/product-detail/Low-Dropout-Regulators-LDO_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; MOQ (none) -> 1; MPN (none) -> AMS1117-3.3; Manufacturer (none) -> Advanced Monolithic Systems; Price (none) -> 0.14; VPN (none) -> C6186; Vendor (none) -> LCSC
Connections:
- net +3.3V: now also R40.1, R41.2
- net D4-SDA: now also R40.2
- net D5-SCL: now also R41.1
- net GND: now also J5.1 (Pin_1); no longer J5.2 (Pin_2)
- net at Q19.2 (S): now also J5.2 (Pin_2); no longer J5.1 (Pin_1)
Other:
- moved on the sheet: C2, C3, J5, Q19, U3

Commit message: Development v.2.0
Parts:
- removed R16, R17, R26, R27, R37, R46, R5, R6: 10K, Resistor_SMD:R_0805_2012Metric, symbol Device:R
- added Q20, Q21, Q22, Q23, Q24, Q25, Q26, Q27: NMOS_YJL03N06A, Package_TO_SOT_SMD:SOT-23, symbol Device:Q_NMOS_GSD
Connections:
- net +3.3V: now also R18.2, R19.1, R28.1, R29.1, R38.1, R47.1, R7.1, R8.1
- net GND: now also Q20.2 (S), Q21.2 (S), Q22.2 (S), Q23.2 (S), Q24.2 (S), Q25.2 (S), Q26.2 (S), Q27.2 (S); no longer D10.1 (K), D12.1 (K), D14.1 (K), D16.1 (K), D2.1 (K), D4.1 (K), D7.1 (K), D8.1 (K)
- net P0: now also Q20.1 (G); no longer R7.1
- net P1: now also Q23.1 (G); no longer R19.1
- net P2: now also Q25.1 (G); no longer R29.1
- net P3: now also Q26.1 (G); no longer R38.1
- net P4: now also Q27.1 (G); no longer R47.1
- net P5: now also Q21.1 (G); no longer R8.1
- net P6: now also Q22.1 (G); no longer R18.1
- net P7: now also Q24.1 (G); no longer R28.1
- net at D7.2 (A): now also R18.1; no longer R18.2
- new net: D2.1 (K), Q20.3 (D)
- new net: D8.1 (K), Q23.3 (D)
- new net: D12.1 (K), Q25.3 (D)
- new net: D14.1 (K), Q26.3 (D)
- new net: D16.1 (K), Q27.3 (D)
- new net: D4.1 (K), Q21.3 (D)
- new net: D7.1 (K), Q22.3 (D)
- new net: D10.1 (K), Q24.3 (D)
Other:
- moved on the sheet: D10, D12, D14, D16, D2, D4, D7, D8, R18, R19, R28, R29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
